Commit message: Added my own Braccio IK. Messy files though

File: braccio_arduino_ros_rviz/urdf/braccio_arm.urdf (robot description, URDF)
Before this commit: robot braccio, 8 links, 7 joints
Joints:
- joint base_joint: limit lower=0.0 upper=3.1416 effort=1000.0 velocity=1.0 -> lower=-1.5707 upper=1.5707 effort=1000.0 velocity=1.0

Commit message: Added random inertias to urdf (for gazebo)

File: braccio_arduino_ros_rviz/urdf/braccio_arm.urdf (robot description, URDF)
Before this commit: robot braccio, 8 links, 7 joints
Links:
- link base_link: mass None -> 5
- link braccio_base_link: mass None -> 5
- link elbow_link: mass None -> 5
- link left_gripper_link: mass None -> 5
- link right_gripper_link: mass None -> 5
- link shoulder_link: mass None -> 5
- link wrist_pitch_link: mass None -> 5
- link wrist_roll_link: mass None -> 5
